File: light_remote_controller.kicad_sch (KiCad schematic)
At the start: 33 parts, among them J10 Screw_Terminal_01x02, J11 Screw_Terminal_01x02, J13 Screen, J4 Screw_Terminal_01x02, J5 Screw_Terminal_01x02, J6 Screw_Terminal_01x02, J7 Screw_Terminal_01x02, J8 Screw_Terminal_01x02, J9 Screw_Terminal_01x02, U1 NodeMCU_ESP12E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

Commit message: Final version that went to production
Parts:
- added J14: Screw_Terminal_01x02, TerminalBlock:TerminalBlock_bornier-2_P5.08mm, symbol Connector:Screw_Terminal_01x02
Connections:
- net BTN_WIFI: now also J14.1 (Pin_1)
- net GND: now also J14.2 (Pin_2)
Other:
- moved on the sheet: J12, J2
Changed lines of the file:
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@@
   (title_block
     (title "Light Remote Controller")
+    (date "2022-05-06")
     (rev "v0.1")
     (company "By Luís Pereira")
@@
   (no_connect (at 35.56 27.94))
   (no_connect (at 45.72 109.22))
-  (no_connect (at 166.37 135.89))
+  (no_connect (at 166.37 132.08))
   (no_connect (at 27.94 48.26))
   (no_connect (at 25.4 101.6))
@@
     (stroke (width 0) (type default) (color 0 0 0 0))
   )
-  (wire (pts (xy 162.56 138.43) (xy 166.37 138.43))
+  (wire (pts (xy 162.56 134.62) (xy 166.37 134.62))
+    (stroke (width 0) (type default) (color 0 0 0 0))
+  )
+  (wire (pts (xy 162.56 154.94) (xy 165.1 154.94))
     (stroke (width 0) (type default) (color 0 0 0 0))
   )
@@
     (stroke (width 0) (type default) (color 0 0 0 0))
   )
-  (wire (pts (xy 162.56 147.32) (xy 166.37 147.32))
+  (wire (pts (xy 162.56 143.51) (xy 166.37 143.51))
     (stroke (width 0) (type default) (color 0 0 0 0))
   )
@@
     (stroke (width 0) (type default) (color 0 0 0 0))
   )
-  (wire (pts (xy 162.56 149.86) (xy 166.37 149.86))
+  (wire (pts (xy 162.56 146.05) (xy 166.37 146.05))
     (stroke (width 0) (type default) (color 0 0 0 0))
   )
@@
     (stroke (width 0) (type default) (color 0 0 0 0))
   )
-  (wire (pts (xy 162.56 140.97) (xy 166.37 140.97))
+  (wire (pts (xy 162.56 137.16) (xy 166.37 137.16))
     (stroke (width 0) (type default) (color 0 0 0 0))
   )
@@
     (stroke (width 0) (type default) (color 0 0 0 0))
   )
+  (wire (pts (xy 162.56 152.4) (xy 165.1 152.4))
+    (stroke (width 0) (type default) (color 0 0 0 0))
+  )
   (wire (pts (xy 167.64 66.04) (xy 168.91 66.04))
     (stroke (width 0) (type default) (color 0 0 0 0))
@@
     (effects (font (size 1.27 1.27)) (justify right bottom))
   )
-  (label "POWER_SAVING" (at 162.56 138.43 180)
+  (label "POWER_SAVING" (at 162.56 134.62 180)
     (effects (font (size 1.27 1.27)) (justify right bottom))
   )
@@
     (effects (font (size 1.27 1.27)) (justify right bottom))
   )
-  (label "GND" (at 162.56 140.97 180)
+  (label "GND" (at 162.56 137.16 180)
     (effects (font (size 1.27 1.27)) (justify right bottom))
   )
@@
     (effects (font (size 1.27 1.27)) (justify right bottom))
   )
+  (label "BTN_WIFI" (at 162.56 152.4 180)
+    (effects (font (size 1.27 1.27)) (justify right bottom))
+  )
   (label "GND" (at 82.55 173.99 180)
     (effects (font (size 1.27 1.27)) (justify right bottom))
@@
     (effects (font (size 1.27 1.27)) (justify right bottom))
   )
+  (label "GND" (at 162.56 154.94 180)
+    (effects (font (size 1.27 1.27)) (justify right bottom))
+  )
   (label "I2C_SDA" (at 148.59 172.72 0)
     (effects (font (size 1.27 1.27)) (justify left bottom))
@@
     (effects (font (size 1.27 1.27)) (justify right bottom))
   )
-  (label "GND" (at 162.56 149.86 180)
+  (label "GND" (at 162.56 146.05 180)
     (effects (font (size 1.27 1.27)) (justify right bottom))
   )
@@
     (effects (font (size 1.27 1.27)) (justify right bottom))
   )
-  (label "BTN_WIFI" (at 162.56 147.32 180)
+  (label "BTN_WIFI" (at 162.56 143.51 180)
     (effects (font (size 1.27 1.27)) (justify right bottom))
   )
@@
     (pin "2")
   )
-  (symbol (lib_id "Connector:Conn_01x02_Female") (at 171.45 147.32 0) (unit 1)
-    (in_bom yes) (on_board yes) (fields_autoplaced)
-    (property "Reference" "J12" (id 0) (at 172.1612 147.7553 0)
-      (effects (font (size 1.27 1.27)) (justify left))
-    )
-    (property "Value" "" (id 1) (at 172.1612 150.2922 0)
-      (effects (font (size 1.27 1.27)) (justify left))
-    )
-    (property "Footprint" "" (id 2) (at 171.45 147.32 0)
-      (effects (font (size 1.27 1.27)) hide)
-    )
-    (property "Datasheet" "~" (id 3) (at 171.45 147.32 0)
+  (symbol (lib_id "Connector:Conn_01x02_Female") (at 171.45 143.51 0) (unit 1)
+    (in_bom yes) (on_board yes) (fields_autoplaced)
+    (property "Reference" "J12" (id 0) (at 172.1612 143.9453 0)
+      (effects (font (size 1.27 1.27)) (justify left))
+    )
+    (property "Value" "" (id 1) (at 172.1612 146.4822 0)
+      (effects (font (size 1.27 1.27)) (justify left))
+    )
+    (property "Footprint" "" (id 2) (at 171.45 143.51 0)
+      (effects (font (size 1.27 1.27)) hide)
+    )
+    (property "Datasheet" "~" (id 3) (at 171.45 143.51 0)
       (effects (font (size 1.27 1.27)) hide)
     )
@@
     (pin "2")
   )
+  (symbol (lib_id "Connector:Screw_Terminal_01x02") (at 170.18 152.4 0) (unit 1)
+    (in_bom yes) (on_board yes) (fields_autoplaced)
+    (property "Reference" "J14" (id 0) (at 172.212 152.8353 0)
+      (effects (font (size 1.27 1.27)) (justify left))
+    )
+    (property "Value" "Screw_Terminal_01x02" (id 1) (at 172.212 155.3722 0)
+      (effects (font (size 1.27 1.27)) (justify left))
+    )
+    (property "Footprint" "TerminalBlock:TerminalBlock_bornier-2_P5.08mm" (id 2) (at 170.18 152.4 0)
+      (effects (font (size 1.27 1.27)) hide)
+    )
+    (property "Datasheet" "~" (id 3) (at 170.18 152.4 0)
+      (effects (font (size 1.27 1.27)) hide)
+    )
+    (pin "1")
+    (pin "2")
+  )
   (symbol (lib_id "Device:R") (at 167.64 50.8 180) (unit 1)
     (in_bom yes) (on_board yes)
@@
     (pin "2")
   )
-  (symbol (lib_id "Connector:Conn_01x03_Female") (at 171.45 138.43 0) (unit 1)
-    (in_bom yes) (on_board yes) (fields_autoplaced)
-    (property "Reference" "J2" (id 0) (at 172.1612 137.5953 0)
-      (effects (font (size 1.27 1.27)) (justify left))
-    )
-    (property "Value" "" (id 1) (at 172.1612 140.1322 0)
-      (effects (font (size 1.27 1.27)) (justify left))
-    )
-    (property "Footprint" "" (id 2) (at 171.45 138.43 0)
-      (effects (font (size 1.27 1.27)) hide)
-    )
-    (property "Datasheet" "~" (id 3) (at 171.45 138.43 0)
+  (symbol (lib_id "Connector:Conn_01x03_Female") (at 171.45 134.62 0) (unit 1)
+    (in_bom yes) (on_board yes) (fields_autoplaced)
+    (property "Reference" "J2" (id 0) (at 172.1612 133.7853 0)
+      (effects (font (size 1.27 1.27)) (justify left))
+    )
+    (property "Value" "" (id 1) (at 172.1612 136.3222 0)
+      (effects (font (size 1.27 1.27)) (justify left))
+    )
+    (property "Footprint" "" (id 2) (at 171.45 134.62 0)
+      (effects (font (size 1.27 1.27)) hide)
+    )
+    (property "Datasheet" "~" (id 3) (at 171.45 134.62 0)
       (effects (font (size 1.27 1.27)) hide)
     )
@@
       (reference "J13") (unit 1) (value "Screen") (footprint "TerminalBlock:TerminalBlock_bornier-4_P5.08mm")
     )
+    (path "/b3807a8d-fc63-426a-b208-4b5a836f3228"
+      (reference "J14") (unit 1) (value "Screw_Terminal_01x02") (footprint "TerminalBlock:TerminalBlock_bornier-2_P5.08mm")
+    )
     (path "/356d8587-2bd3-4816-9283-b56463cc4546"
